Commit message: fix: spider.urdf 다리 배치 변경에 따른 gait 파라미터 재매핑
- spider.urdf: 다리 배치 변경 (A=FR, B=BR, C=FL, D=BL)
  - foot 링크에 inertial, collision 추가 (loadURDF 오류 수정)
  - foot 조인트에 limit 추가 (REVOLUTE limit 경고 수정)
  - XML 태그 오류 수정
- walk_sim.py / trot_sim.py: PHY_CONTACT, ARM_DIR, SWING_START 재매핑

Co-Authored-By: Claude Sonnet 4.6 <noreply@anthropic.com>

File: simulation/spider.urdf (robot description, URDF)
Before this commit: robot spider, 9 links, 8 joints
Joints:
- joint arm_a: origin xyz=-0.06 0.06 0 rpy=0 0 2.3562 -> xyz=0.06 0.06 0 rpy=0 0 0.7854
- joint arm_b: origin xyz=0.06 0.06 0 rpy=0 0 0.7854 -> xyz=0.06 -0.06 0 rpy=0 0 -0.7854
- joint arm_c: origin xyz=-0.06 -0.06 0 rpy=0 0 -2.3562 -> xyz=-0.06 0.06 0 rpy=0 0 2.3562
- joint arm_d: origin xyz=0.06 -0.06 0 rpy=0 0 -0.7854 -> xyz=-0.06 -0.06 0 rpy=0 0 -2.3562
